Commit message: Modularização dos arquivos .xacro e .gazebo

File: RobotTraining_P3dx_Gazebo/p3dx_description_gazebo/urdf/pioneer3dx.xacro (robot description, xacro)
@@ -22,9 +22,35 @@
 	<!-- import the pioneer 3dx's wheels -->
 	<xacro:include filename="$(find p3dx_description_gazebo)/urdf/pioneer3dx_wheel.xacro" />
-	<!-- chassis -->
+	<!-- import imu -->
+	<xacro:include filename="$(find p3dx_description_gazebo)/urdf/sensors/imu/imu.xacro"/>
+	<xacro:include filename="$(find p3dx_description_gazebo)/urdf/sensors/imu/imu.gazebo"/>
+	<!-- import ground truth -->
+	<xacro:include filename="$(find p3dx_description_gazebo)/urdf/sensors/groundTruth/groundTruth.gazebo"/>
+	<!-- import odometry -->
+	<xacro:include filename="$(find p3dx_description_gazebo)/urdf/sensors/odometry/odometry.gazebo"/>
+	<!-- import chassis -->
+	<xacro:include filename="$(find p3dx_description_gazebo)/urdf/parts/chassi/chassi.xacro"/>
+	<xacro:include filename="$(find p3dx_description_gazebo)/urdf/parts/chassi/chassi.gazebo"/>
+	<!-- import swivel -->
+	<xacro:include filename="$(find p3dx_description_gazebo)/urdf/parts/swivel/swivel.xacro"/>
+	<xacro:include filename="$(find p3dx_description_gazebo)/urdf/parts/swivel/swivel.gazebo"/>
+	<!-- import top_plate -->
+	<xacro:include filename="$(find p3dx_description_gazebo)/urdf/parts/top_plate/top_plate.xacro"/>
+	<xacro:include filename="$(find p3dx_description_gazebo)/urdf/parts/top_plate/top_plate.gazebo"/>
+	<!-- import center_hubcap -->
+	<xacro:include filename="$(find p3dx_description_gazebo)/urdf/parts/center_hubcap/center_hubcap.xacro"/>
+	<xacro:include filename="$(find p3dx_description_gazebo)/urdf/parts/center_hubcap/center_hubcap.gazebo"/>
+	<!-- import center_wheel -->
+	<xacro:include filename="$(find p3dx_description_gazebo)/urdf/parts/center_wheel/center_wheel.xacro"/>
+	<xacro:include filename="$(find p3dx_description_gazebo)/urdf/parts/center_wheel/center_wheel.gazebo"/>
+	<xacro:p3dx_wheel suffix="left" parent="base_link" reflect="-1"/>
+	<xacro:p3dx_wheel suffix="right" parent="base_link" reflect="1"/>
+	<!-- import front_sonar -->
+	<xacro:include filename="$(find p3dx_description_gazebo)/urdf/parts/front_sonar/front_sonar.xacro"/>
+	<xacro:include filename="$(find p3dx_description_gazebo)/urdf/parts/front_sonar/front_sonar.gazebo"/>
+	<!-- chassis
 	<link name="base_link">
 		<inertial>
 			<mass value="3.5" />
-			<!--<origin xyz="-0.025 0 -0.223"/> -->
 			<origin xyz="-0.05 0 0" />
 			<inertia ixx="1" ixy="0" ixz="0" iyy="1" iyz="0" izz="1" />
@@ -45,6 +71,6 @@
 			</geometry>
 		</collision>
-	</link>
-	<!-- top_plate -->
+	</link>-->
+	<!-- top_plate
 	<link name="top_plate">
 		<inertial>
@@ -73,6 +99,6 @@
 		<parent link="base_link" />
 		<child link="top_plate" />
-	</joint>
-	<!-- swivel -->
+	</joint>-->
+	<!-- swivel
 	<link name="swivel">
 		<inertial>
@@ -105,6 +131,6 @@
 		<parent link="base_link" />
 		<child link="swivel" />
-	</joint>
-	<!-- center_hubcap -->
+	</joint>-->
+	<!-- center_hubcap
 	<link name="center_hubcap">
 		<inertial>
@@ -137,6 +163,6 @@
 		<parent link="swivel" />
 		<child link="center_wheel" />
-	</joint>
-	<!-- center_wheel -->
+	</joint> -->
+	<!-- center_wheel
 	<link name="center_wheel">
 		<inertial>
@@ -165,5 +191,5 @@
 		<parent link="center_wheel"/>
 		<child link="center_hubcap"/>
-	</joint>
+	</joint>-->
 	<!-- End of Legacy for diff drive plugin
 	https://github.com/ros-simulation/gazebo_ros_pkgs/pull/707/files
@@ -172,7 +198,5 @@
 	"To fix an old package you have to exchange left wheel by the right wheel.\n"
 	-->
-	<xacro:p3dx_wheel suffix="left" parent="base_link" reflect="-1"/>
-	<xacro:p3dx_wheel suffix="right" parent="base_link" reflect="1"/>
-	<!-- front_sonar -->
+	<!-- front_sonar
 	<link name="front_sonar">
 		<inertial>
@@ -201,5 +225,5 @@
 		<parent link="base_link" />
 		<child link="front_sonar" />
-	</joint>
+	</joint>-->
 	<!-- lms100 laser -->
 	<link name="lms100">
@@ -228,5 +252,5 @@
 		<child link="lms100" />
 	</joint>
-	<!-- IMU -->
+	<!-- IMU
 	<link name="base_IMU">
 		<collision>
@@ -253,5 +277,5 @@
 		<parent link="base_link"/>
 		<child link="base_IMU"/>
-	</joint>
+	</joint>-->
 	<link name="base_Cam">
 		<collision>

Commit message: Modularização dos arquivos .xacro e .gazebo

File: RobotTraining_P3dx_Gazebo/p3dx_description_gazebo/urdf/pioneer3dx.xacro (robot description, xacro)
@@ -29,4 +29,17 @@
 	<!-- import odometry -->
 	<xacro:include filename="$(find p3dx_description_gazebo)/urdf/sensors/odometry/odometry.gazebo"/>
+	<!-- import camera -->
+	<xacro:include filename="$(find p3dx_description_gazebo)/urdf/sensors/camera/camera.xacro"/>
+	<xacro:include filename="$(find p3dx_description_gazebo)/urdf/sensors/camera/camera.gazebo"/>
+	<!-- import sonar -->
+	<!-- import sonar_1 -->
+	<xacro:include filename="$(find p3dx_description_gazebo)/urdf/sensors/sonar/sonar_1.xacro"/>
+	<xacro:include filename="$(find p3dx_description_gazebo)/urdf/sensors/sonar/sonar_1.gazebo"/>
+	<!-- import sonar_2 -->
+	<xacro:include filename="$(find p3dx_description_gazebo)/urdf/sensors/sonar/sonar_2.xacro"/>
+	<xacro:include filename="$(find p3dx_description_gazebo)/urdf/sensors/sonar/sonar_2.gazebo"/>
+	<!-- import sonar_3 -->
+	<xacro:include filename="$(find p3dx_description_gazebo)/urdf/sensors/sonar/sonar_3.xacro"/>
+	<xacro:include filename="$(find p3dx_description_gazebo)/urdf/sensors/sonar/sonar_3.gazebo"/>
 	<!-- import chassis -->
 	<xacro:include filename="$(find p3dx_description_gazebo)/urdf/parts/chassi/chassi.xacro"/>
@@ -277,5 +290,5 @@
 		<parent link="base_link"/>
 		<child link="base_IMU"/>
-	</joint>-->
+	</joint>
 	<link name="base_Cam">
 		<collision>
@@ -377,4 +390,4 @@
 		<parent link="base_link"/>
 		<child link="base_sonar_3"/>
-	</joint>
+	</joint>-->
 </robot>

Commit message: Modularização do LiDAR, implementaço do laser scan matcher, correções sonar

File: RobotTraining_P3dx_Gazebo/p3dx_description_gazebo/urdf/pioneer3dx.xacro (robot description, xacro)
@@ -19,5 +19,5 @@
 	xmlns:xacro="http://ros.org/wiki/xacro">
 	<!-- import all gazebo-customization elements, including gazebo colors -->
-	<xacro:include filename="$(find p3dx_description_gazebo)/urdf/pioneer3dx.gazebo" />
+	<!--<xacro:include filename="$(find p3dx_description_gazebo)/urdf/pioneer3dx.gazebo" />-->
 	<!-- import the pioneer 3dx's wheels -->
 	<xacro:include filename="$(find p3dx_description_gazebo)/urdf/pioneer3dx_wheel.xacro" />
@@ -29,4 +29,7 @@
 	<!-- import odometry -->
 	<xacro:include filename="$(find p3dx_description_gazebo)/urdf/sensors/odometry/odometry.gazebo"/>
+	<!-- import LiDAR-->
+	<xacro:include filename="$(find p3dx_description_gazebo)/urdf/sensors/lidar/lidar.xacro"/>
+	<xacro:include filename="$(find p3dx_description_gazebo)/urdf/sensors/lidar/lidar.gazebo"/>
 	<!-- import camera -->
 	<xacro:include filename="$(find p3dx_description_gazebo)/urdf/sensors/camera/camera.xacro"/>
@@ -62,332 +65,3 @@
 	<xacro:include filename="$(find p3dx_description_gazebo)/urdf/parts/front_sonar/front_sonar.xacro"/>
 	<xacro:include filename="$(find p3dx_description_gazebo)/urdf/parts/front_sonar/front_sonar.gazebo"/>
-	<!-- chassis
-	<link name="base_link">
-		<inertial>
-			<mass value="3.5" />
-			<origin xyz="-0.05 0 0" />
-			<inertia ixx="1" ixy="0" ixz="0" iyy="1" iyz="0" izz="1" />
-		</inertial>
-		<visual>
-			<origin xyz="-0.045 0 0.148" rpy="0 0 0" />
-			<geometry name="pioneer_geom">
-				<mesh filename="package://p3dx_description_gazebo/meshes/chassis.stl" />
-			</geometry>
-			<material name="ChassisRed">
-				<color rgba="0.851 0.0 0.0 1.0" />
-			</material>
-		</visual>
-		<collision>
-			<origin xyz="-0.045 0 0.145" rpy="0 0 0" />
-			<geometry>
-				<box size="0.35 0.25 0.14" />
-			</geometry>
-		</collision>
-	</link>-->
-	<!-- top_plate
-	<link name="top_plate">
-		<inertial>
-			<mass value="0.01" />
-			<origin xyz="0 0 0" />
-			<inertia ixx="1" ixy="0" ixz="0" iyy="1" iyz="0" izz="1" />
-		</inertial>
-		<visual>
-			<origin xyz="0 0 0" rpy="0 0 0" />
-			<geometry name="top_geom">
-				<mesh filename="package://p3dx_description_gazebo/meshes/top.stl" />
-			</geometry>
-			<material name="TopBlack">
-				<color rgba="0.038 0.038 0.038 1.0" />
-			</material>
-		</visual>
-		<collision>
-			<origin xyz="0.0 0 0" rpy="0 0 0" />
-			<geometry name="pioneer_geom">
-				<box size="0.45 0.38 0.01" />
-			</geometry>
-		</collision>
-	</link>
-	<joint name="base_top_joint" type="fixed">
-		<origin xyz="-0.045 0 0.234" rpy="0 0 0" />
-		<parent link="base_link" />
-		<child link="top_plate" />
-	</joint>-->
-	<!-- swivel
-	<link name="swivel">
-		<inertial>
-			<mass value="0.1" />
-			<origin xyz="0 0 0" />
-			<inertia ixx="0.01" ixy="0" ixz="0" iyy="0.01" iyz="0" izz="0.01" />
-		</inertial>
-		<visual>
-			<origin xyz="0 0 0" rpy="0 0 0" />
-			<geometry name="pioneer_geom">
-				<mesh filename="package://p3dx_description_gazebo/meshes/swivel.stl" />
-			</geometry>
-			<material name="swivel">
-				<color rgba="0.5 0.5 0.5 1" />
-			</material>
-		</visual>
-		<collision>
-			<origin xyz="0 0 0" rpy="0 0 0" />
-			<geometry>
-				<box size="0.00001 0.00001 0.00001" />
-			</geometry>
-		</collision>
-	</link>
-	<joint name="base_swivel_joint" type="fixed">
-		<origin xyz="-0.185 0 0.055" rpy="0 0 0" />
-		<axis xyz="0 0 1" />
-		<anchor xyz="0 0 0" />
-		<limit effort="100" velocity="100" k_velocity="0" />
-		<joint_properties damping="0.0" friction="0.0" />
-		<parent link="base_link" />
-		<child link="swivel" />
-	</joint>-->
-	<!-- center_hubcap
-	<link name="center_hubcap">
-		<inertial>
-			<mass value="0.01" />
-			<origin xyz="0 0 0" />
-			<inertia ixx="0.012411765597" ixy="-0.000711733678" ixz="0.00050272983" iyy="0.015218160428" iyz="-0.000004273467" izz="0.011763977943" />
-		</inertial>
-		<visual>
-			<origin xyz="0 0 0" rpy="0 0 0" />
-			<geometry name="pioneer_geom">
-				<mesh filename="package://p3dx_description_gazebo/meshes/center_hubcap.stl" />
-			</geometry>
-			<material name="swivel">
-				<color rgba="0.5 0.5 0.5 1" />
-			</material>
-		</visual>
-		<collision>
-			<origin xyz="0 0 0" rpy="0 0 0" />
-			<geometry>
-				<box size="0.00001 0.00001 0.00001" />
-			</geometry>
-		</collision>
-	</link>
-	<joint name="swivel_hubcap_joint" type="fixed">
-		<origin xyz="-0.026 0 -0.016" rpy="0 0 0" />
-		<axis xyz="0 1 0" />
-		<anchor xyz="0 0 0" />
-		<limit effort="100" velocity="100" k_velocity="0" />
-		<joint_properties damping="0.0" friction="0.0" />
-		<parent link="swivel" />
-		<child link="center_wheel" />
-	</joint> -->
-	<!-- center_wheel
-	<link name="center_wheel">
-		<inertial>
-			<mass value="1.0" />
-			<origin xyz="0 0 0" />
-			<inertia ixx="0.012411765597" ixy="-0.000711733678" ixz="0.00050272983" iyy="0.015218160428" iyz="-0.000004273467" izz="0.011763977943" />
-		</inertial>
-		<visual>
-			<origin xyz="0 0 0" rpy="0 0 0" />
-			<geometry name="pioneer_geom">
-				<mesh filename="package://p3dx_description_gazebo/meshes/center_wheel.stl" />
-			</geometry>
-			<material name="WheelBlack">
-				<color rgba="0.117 0.117 0.117 1" />
-			</material>
-		</visual>
-		<collision>
-			<origin xyz="0 0 0" rpy="${-3.1415927/2.0} 0 0" />
-			<geometry>
-				<cylinder radius="0.0375" length="0.01" />
-			</geometry>
-		</collision>
-	</link>
-	<joint name="center_wheel_joint" type="fixed">
-		<origin xyz="-0.0035 0 -0.001" rpy="0 0 0"/>
-		<parent link="center_wheel"/>
-		<child link="center_hubcap"/>
-	</joint>-->
-	<!-- End of Legacy for diff drive plugin
-	https://github.com/ros-simulation/gazebo_ros_pkgs/pull/707/files
-	"This setting assumes you have a old package, where the right and left wheel are changed to fix a former code issue\n"
-	"To get rid of this error just set <legacyMode> to false if you just created a new package.\n"
-	"To fix an old package you have to exchange left wheel by the right wheel.\n"
-	-->
-	<!-- front_sonar
-	<link name="front_sonar">
-		<inertial>
-			<mass value="0.0001" />
-			<origin xyz="0 0 0" />
-			<inertia ixx="1" ixy="0" ixz="0" iyy="1" iyz="0" izz="1" />
-		</inertial>
-		<visual>
-			<origin rpy="0 0 0" xyz="0 0 0" />
-			<geometry name="pioneer_geom">
-				<mesh filename="package://p3dx_description_gazebo/meshes/front_sonar.stl" />
-			</geometry>
-			<material name="SonarYellow">
-				<color rgba="0.715 0.583 0.210 1.0" />
-			</material>
-		</visual>
-		<collision>
-			<origin rpy="0 0 0" xyz="0 0 0" />
-			<geometry>
-				<box size="0.00001 0.00001 0.00001" />
-			</geometry>
-		</collision>
-	</link>
-	<joint name="base_front_joint" type="fixed">
-		<origin rpy="0 0 0" xyz="0.109 0 0.209" />
-		<parent link="base_link" />
-		<child link="front_sonar" />
-	</joint>-->
-	<!-- lms100 laser -->
-	<link name="lms100">
-		<inertial>
-			<mass value="1e-5" />
-			<origin xyz="0 0 0" rpy="0 0 0" />
-			<inertia ixx="1e-6" ixy="0" ixz="0" iyy="1e-6" iyz="0" izz="1e-6" />
-		</inertial>
-		<visual>
-			<origin xyz="0 0 0" rpy="0 0 0" />
-			<geometry>
-				<mesh filename="package://p3dx_description_gazebo/meshes/lms100.dae" />
-			</geometry>
-		</visual>
-		<collision>
-			<origin xyz="0 0 0" rpy="0 0 0" />
-			<geometry>
-				<box size="0.1 0.1 0.1" />
-			</geometry>
-		</collision>
-	</link>
-	<joint name="lms100_joint" type="fixed">
-		<axis xyz="0 1 0" />
-		<origin xyz="0.16 0 0.15" rpy="0 0 0" />
-		<parent link="base_link" />
-		<child link="lms100" />
-	</joint>
-	<!-- IMU
-	<link name="base_IMU">
-		<collision>
-			<origin xyz="0 0 0" rpy="0 0 0"/>
-			<geometry>
-			<box size="0.0 0.0 0.0"/>
-			</geometry>
-		</collision>
-		<visual>
-			<origin xyz="0 0 0" rpy="0 0 0"/>
-			<geometry>
-				<box size="0.01 0.01 0.01"/>
-			</geometry>
-		</visual>
-		<inertial>
-			<mass value="1e-5" />
-			<origin xyz="0 0 0" rpy="0 0 0"/>
-			<inertia ixx="1e-6" ixy="0" ixz="0" iyy="1e-6" iyz="0"      izz="1e-6" />
-		</inertial>
-	</link>
-	<joint name="IMU_joint" type="fixed">
-		<axis xyz="0 1 0" />
-		<origin rpy="0 0 0" xyz="0 0 0.09" />
-		<parent link="base_link"/>
-		<child link="base_IMU"/>
-	</joint>
-	<link name="base_Cam">
-		<collision>
-			<origin xyz="0 0 0" rpy="0 0 0"/>
-			<geometry>
-			<box size="0.01 0.01 0.01"/>
-			</geometry>
-		</collision>
-		<visual>
-			<origin xyz="0 0 0" rpy="0 0 0"/>
-			<geometry>
-				<mesh filename="package://p3dx_description_gazebo/meshes/kinect.dae" />
-			</geometry>
-		</visual>
-		<inertial>,
-			<mass value="1e-5" />
-			<origin xyz="0 0 0" rpy="0 0 0"/>
-			<inertia ixx="1e-6" ixy="0" ixz="0" iyy="1e-6" iyz="0"      izz="1e-6" />
-		</inertial>
-	</link>
-	<joint name="Cam_joint" type="fixed">
-		<axis xyz="0 1 0" />
-		<origin xyz="0.12 0 0.28" rpy="0 0 0" />
-		<parent link="base_link"/>
-		<child link="base_Cam"/>
-	</joint>
-	<link name="base_sonar_1">
-		<collision>
-		<origin xyz="0 0 0" rpy="0 0 0"/>
-		<geometry>
-			<box size="0.01 0.01 0.01"/>
-		</geometry>
-		</collision>
-		<visual>
-		<origin xyz="0 0 0" rpy="0 0 0"/>
-		<geometry>
-			<box size="0.01 0.01 0.01"/>
-		</geometry>
-		</visual>
-		<inertial>
-		<mass value="1e-5" />
-		<origin xyz="0 0 0" rpy="0 0 0"/>
-		<inertia ixx="1e-6" ixy="0" ixz="0" iyy="1e-6" iyz="0"      izz="1e-6" />
-		</inertial>
-	</link>
-	<joint name="Sonar_1_joint" type="fixed">
-		<axis xyz="0 1 0" />
-		<origin xyz="0.08 -0.12 0.2" rpy="0 0 -1.57" />
-		<parent link="base_link"/>
-		<child link="base_sonar_1"/>
-	</joint>
-	<link name="base_sonar_2">
-		<collision>
-		<origin xyz="0 0 0" rpy="0 0 0"/>
-		<geometry>
-			<box size="0.01 0.01 0.01"/>
-		</geometry>
-		</collision>
-		<visual>
-		<origin xyz="0 0 0" rpy="0 0 0"/>
-		<geometry>
-			<box size="0.01 0.01 0.01"/>
-		</geometry>
-		</visual>
-		<inertial>
-		<mass value="1e-5" />
-		<origin xyz="0 0 0" rpy="0 0 0"/>
-		<inertia ixx="1e-6" ixy="0" ixz="0" iyy="1e-6" iyz="0"      izz="1e-6" />
-		</inertial>
-	</link>
-	<joint name="Sonar_2_joint" type="fixed">
-		<axis xyz="0 1 0" />
-		<origin xyz="0.16 0 0.21" rpy="0 0 0" />
-		<parent link="base_link"/>
-		<child link="base_sonar_2"/>
-	</joint>
-	<link name="base_sonar_3">
-		<collision>
-		<origin xyz="0 0 0" rpy="0 0 0"/>
-		<geometry>
-			<box size="0.01 0.01 0.01"/>
-		</geometry>
-		</collision>
-		<visual>
-		<origin xyz="0 0 0" rpy="0 0 0"/>
-		<geometry>
-			<box size="0.01 0.01 0.01"/>
-		</geometry>
-		</visual>
-		<inertial>
-		<mass value="1e-5" />
-		<origin xyz="0 0 0" rpy="0 0 0"/>
-		<inertia ixx="1e-6" ixy="0" ixz="0" iyy="1e-6" iyz="0"      izz="1e-6" />
-		</inertial>
-	</link>
-	<joint name="Sonar_3_joint" type="fixed">
-		<axis xyz="0 1 0" />
-		<origin xyz="0.08 0.12 0.2" rpy="0 0 1.57" />
-		<parent link="base_link"/>
-		<child link="base_sonar_3"/>
-	</joint>-->
 </robot>
